Commit message: set proper friction

File: elektron_defs/robots/elektron.udrf.xacro (robot description, xacro)
@@ -21,5 +21,6 @@
 			<origin xyz="-0.0 0 0.115" rpy="0 0 0" />
 			<geometry>
-				<mesh filename="package://elektron_defs/meshes/elektron_body.blend"/>
+<box size="0.38 0.28 0.20" />
+				<!--<mesh filename="package://elektron_defs/meshes/elektron_body.blend"/>-->
 			</geometry>
 		</visual>
@@ -43,4 +44,5 @@
 			<parent link="${parent}" />
 			<child link="${parent}_${suffix}_wheel_link" />
+ <dynamics damping="0.0" friction="0.0"/>
 		</joint>
 		<link name="${parent}_${suffix}_wheel_link">
@@ -62,20 +64,53 @@
 					<cylinder radius="${wheel_radius}" length="${wheel_length}" />
 				</geometry>
+<!-- <surface>
+            <friction>
+              <ode>
+                <mu>${m}</mu>
+                <mu2>${m}</mu2>
+                <fdir1>1.000000 0.000000 0.000000</fdir1>
+                <slip1>10000.000000</slip1>
+                <slip2>10000.000000</slip2>
+              </ode>
+            </friction>
+            <bounce>
+              <restitution_coefficient>0.000000</restitution_coefficient>
+              <threshold>100000.000000</threshold>
+            </bounce>
+            <contact>
+              <ode>
+                <soft_cfm>0.000000</soft_cfm>
+                <soft_erp>0.200000</soft_erp>
+                <kp>100000.000000</kp>
+                <kd>1.000000</kd>
+                <max_vel>100.000000</max_vel>
+                <min_depth>0.001000</min_depth>
+              </ode>
+            </contact>
+          </surface> -->
 			</collision>
 		</link>
-		<gazebo reference="${parent}_${suffix}_wheel_link" >
+<gazebo reference="${parent}_${suffix}_wheel_link">
+      <mu1 value="${m}" />
+      <mu2 value="${m}" />
+      <kp value="100000.0" />
+      <kd value="0.00001" />
+      <maxVel value="1.0" />
+      <minDepth value="0.0001" />
+    </gazebo>
+	<!--	<gazebo reference="${parent}_${suffix}_wheel_link" >
 			<elem key="mu1" value="${m}" />
 			<elem key="mu2" value="${m}" />
 			<elem key="kp"  value="100000000.0" />
 			<elem key="kd"  value="1.0" />
-		</gazebo>
+		</gazebo> -->
 	</xacro:macro>
-	<xacro:erratic_wheel suffix="left" parent="base_link" reflect="1" offset="0" m="0.1"/>
-	<xacro:erratic_wheel suffix="left_front" parent="base_link" reflect="1" offset="0.15" m="100.1"/>
-	<xacro:erratic_wheel suffix="left_rear" parent="base_link" reflect="1" offset="-0.15" m="100.1"/>
-	<xacro:erratic_wheel suffix="right" parent="base_link" reflect="-1" offset="0" m="0.1"/>
+	<xacro:erratic_wheel suffix="left" parent="base_link" reflect="1" offset="0" m="0.900"/>
+	<xacro:erratic_wheel suffix="left_front" parent="base_link" reflect="1" offset="0.15" m="0"/>
+	<xacro:erratic_wheel suffix="left_rear" parent="base_link" reflect="1" offset="-0.15" m="0"/>
+	<xacro:erratic_wheel suffix="right" parent="base_link" reflect="-1" offset="0" m="0.900"/>
 	<xacro:erratic_wheel suffix="right_front" parent="base_link" reflect="-1" offset="0.15"
-		m="100.1"/>
-	<xacro:erratic_wheel suffix="right_rear" parent="base_link" reflect="-1" offset="-0.15"	m="100.1"/>
+		m="0"/>
+	<xacro:erratic_wheel suffix="right_rear" parent="base_link" reflect="-1" offset="-0.15"	m="0"/>
 	<joint name="base_laser_joint" type="fixed">
 		<origin rpy="0 0 0" xyz="0.14 0 0.3"/>
@@ -127,8 +162,7 @@
 	</gazebo>
 	<gazebo>
-		<controller:diffdrive_plugin name="differential_drive_controller" plugin="libdiffdrive_plugin.so">
-			<alwaysOn>true</alwaysOn>
-			<update>100</update>
-			<updateRate>100.0</updateRate>
+		<plugin name="differential_drive_controller" filename="libgazebo_ros_diff_drive.so">
+			<alwaysOn>true</alwaysOn>
+			<updateRate>100</updateRate>
 			<leftJoint>base_link_right_wheel_joint</leftJoint>
 			<rightJoint>base_link_left_wheel_joint</rightJoint>
@@ -136,8 +170,11 @@
 			<wheelDiameter>${wheel_radius*2}</wheelDiameter>
 			<torque>5</torque>
-			<interface:position name="position_iface_0"/>
-			<robotNamespace>/</robotNamespace>
-			<topicName>cmd_vel</topicName>
-		</controller:diffdrive_plugin>
+			<commandTopic>cmd_vel</commandTopic>
+			<odometryTopic>odom</odometryTopic>
+			<odometryFrame>odom</odometryFrame>
+			<robotBaseFrame>base_link</robotBaseFrame>
+		</plugin>
+	</gazebo>
+	<gazebo>
 		<controller:gazebo_ros_p3d name="p3d_base_controller" plugin="libgazebo_ros_p3d.so">
 			<alwaysOn>true</alwaysOn>

Commit message: add laser model | config laser scans

File: elektron_defs/robots/elektron.udrf.xacro (robot description, xacro)
@@ -21,6 +21,6 @@
 			<origin xyz="-0.0 0 0.115" rpy="0 0 0" />
 			<geometry>
-<box size="0.38 0.28 0.20" />
-				<!--<mesh filename="package://elektron_defs/meshes/elektron_body.blend"/>-->
+<!--<box size="0.38 0.28 0.20" />-->
+				<mesh filename="package://elektron_defs/meshes/elektron_body.dae"/>
 			</geometry>
 		</visual>
@@ -127,5 +127,6 @@
 			<origin rpy="0 0 0" xyz="0 0 0.0"/>
 			<geometry>
-				<box size="0.15 0.15 0.2"/>
+<mesh filename="package://elektron_defs/meshes/sick_lms1xx.dae"/>
+				<!--<box size="0.15 0.15 0.2"/>-->
 			</geometry>
 		</visual>
@@ -137,28 +138,40 @@
 		</collision>
 	</link>
-	<gazebo reference="base_laser_link">
-		<sensor:ray name="base_laser_link">
-			<resRange>0.01</resRange>
-			<rayCount>181</rayCount>
-			<rangeCount>181</rangeCount>
-			<laserCount>1</laserCount>
-			<origin>0.0 0.0 0.0</origin>
-			<displayRays>true</displayRays>
-			<minAngle>-90</minAngle>
-			<maxAngle>90</maxAngle>
-			<minRange>0.07</minRange>
-			<maxRange>10.0</maxRange>
-			<updateRate>25.0</updateRate>
-			<controller:gazebo_ros_laser name="gazebo_ros_base_laser_link_controller"
-				plugin="libgazebo_ros_laser.so">
-				<gaussianNoise>0.005</gaussianNoise>
-				<alwaysOn>true</alwaysOn>
-				<updateRate>25.0</updateRate>
-				<topicName>base_scan</topicName>
-				<frameName>base_laser_link</frameName>
-				<interface:laser name="gazebo_ros_base_laser_link_iface"/>
-			</controller:gazebo_ros_laser>
-		</sensor:ray>
-	</gazebo>
+<!-- hokuyo -->
+  <gazebo reference="base_laser_link">
+   <sensor type="gpu_ray" name="head_hokuyo_sensor">
+      <pose>0 0 0 0 0 0</pose>
+      <visualize>true</visualize>
+      <update_rate>40</update_rate>
+      <ray>
+        <scan>
+          <horizontal>
+            <samples>720</samples>
+            <resolution>1</resolution>
+            <min_angle>-1.570796</min_angle>
+            <max_angle>1.570796</max_angle>
+          </horizontal>
+        </scan>
+        <range>
+          <min>0.10</min>
+          <max>15.0</max>
+          <resolution>0.01</resolution>
+        </range>
+        <noise>
+          <type>gaussian</type>
+          <!-- Noise parameters based on published spec for Hokuyo laser
+               achieving "+-30mm" accuracy at range < 10m.  A mean of 0.0m and
+               stddev of 0.01m will put 99.7% of samples within 0.03m of the true
+               reading. -->
+          <mean>0.0</mean>
+          <stddev>0.01</stddev>
+        </noise>
+      </ray>
+      <plugin name="gazebo_ros_head_hokuyo_controller" filename="libgazebo_ros_gpu_laser.so">
+        <topicName>/laser_scan</topicName>
+        <frameName>base_laser_link</frameName>
+      </plugin>
+    </sensor>
+  </gazebo>
 	<gazebo>
 		<plugin name="differential_drive_controller" filename="libgazebo_ros_diff_drive.so">
